File: Hardware/moduplay/moduplay.kicad_sch (KiCad schematic)
At the start: 0 parts

Commit message: Add basic components
Parts:
- added BT1: Battery, symbol Device:Battery
- added SW1: Left, symbol Switch:SW_Push
- added SW10: Power_Switch, symbol Switch:SW_DIP_x01
- added SW2: Up, symbol Switch:SW_Push
- added SW3: Right, symbol Switch:SW_Push
- added SW4: Down, symbol Switch:SW_Push
- added SW5: X, symbol Switch:SW_Push
- added SW6: Y, symbol Switch:SW_Push
- added SW7: B, symbol Switch:SW_Push
- added SW8: A, symbol Switch:SW_Push
- added SW9: Menu, symbol Switch:SW_Push
Connections:
- new net: BT1.1 (+), SW10.1
- new net GND: BT1.2 (-)
- new net VCC: SW10.2

Commit message: Finish scheme
Parts:
- added DS1: ~, symbol local:OLED12864_SPI_SSD1309
- added J1: ~, symbol local:Edge_Connector
Connections:
- net GND: now also DS1.1 (VSS), J1.29 (GND)
- net VCC: now also DS1.2 (VDD), J1.1 (VCC)
- net at SW3.1: now also J1.20 (BTN_RIGHT2)
- net at SW3.2: now also J1.18 (BTN_RIGHT1)
- net at SW6.1: now also J1.26 (BTN_Y1)
- net at SW6.2: now also J1.28 (BTN_Y2)
- net at SW9.1: now also J1.11 (BTN_MENU2)
- net at SW9.2: now also J1.9 (BTN_MENU1)
- net at SW2.1: now also J1.13 (BTN_UP1)
- net at SW2.2: now also J1.15 (BTN_UP2)
- net at SW1.1: now also J1.19 (BTN_LEFT2)
- net at SW1.2: now also J1.17 (BTN_LEFT1)
- net at SW8.1: now also J1.23 (BTN_A2)
- net at SW8.2: now also J1.21 (BTN_A1)
- net at SW5.1: now also J1.27 (BTN_X2)
- net at SW5.2: now also J1.25 (BTN_X1)
- net at SW4.1: now also J1.14 (BTN_DOWN1)
- net at SW4.2: now also J1.16 (BTN_DOWN2)
- net at SW7.1: now also J1.22 (BTN_B1)
- net at SW7.2: now also J1.24 (BTN_B2)
- new net: DS1.4 (SDA), J1.3 (SCR_SDA)
- new net: DS1.7 (CS), J1.4 (SCR_CS)
- new net: DS1.3 (SCLK), J1.5 (SCR_SCL)
- new net: DS1.5 (RES), J1.6 (SCR_RES)
- new net: DS1.6 (DC), J1.8 (SCR_DC)
- no-connect marks 0 -> 5
Other:
- title: (none) -> ModuPlay main board
- moved on the sheet: BT1, SW1, SW10, SW2, SW3, SW4, SW5, SW6, SW7, SW8, SW9

Commit message: Add buzzer
Parts:
- removed J1: ~, symbol local:Edge_Connector
- added BZ1: Buzzer, symbol Device:Buzzer
- added J1: ~, symbol local:Edge_Connector_Slot
Connections:
- net GND: now also J1.29 (GND)
- net VCC: now also J1.1 (VCC)
- net at SW3.1: now also J1.20 (BTN_RIGHT2)
- net at SW3.2: now also J1.18 (BTN_RIGHT1)
- net at SW6.1: now also J1.26 (BTN_Y1)
- net at SW6.2: now also J1.28 (BTN_Y2)
- net at SW9.1: now also J1.11 (BTN_MENU2)
- net at SW9.2: now also J1.9 (BTN_MENU1)
- net at SW2.1: now also J1.13 (BTN_UP1)
- net at SW4.1: now also J1.14 (BTN_DOWN1)
- net at SW2.2: now also J1.15 (BTN_UP2)
- net at SW4.2: now also J1.16 (BTN_DOWN2)
- net at SW1.2: now also J1.17 (BTN_LEFT1)
- net at SW1.1: now also J1.19 (BTN_LEFT2)
- net at SW8.2: now also J1.21 (BTN_A1)
- net at SW7.1: now also J1.22 (BTN_B1)
- net at SW8.1: now also J1.23 (BTN_A2)
- net at SW7.2: now also J1.24 (BTN_B2)
- net at SW5.2: now also J1.25 (BTN_X1)
- net at SW5.1: now also J1.27 (BTN_X2)
- net at DS1.4 (SDA): now also J1.3 (SCR_SDA)
- net at DS1.7 (CS): now also J1.4 (SCR_CS)
- net at DS1.3 (SCLK): now also J1.5 (SCR_SCL)
- net at DS1.5 (RES): now also J1.6 (SCR_RES)
- net at DS1.6 (DC): now also J1.8 (SCR_DC)
- new net: BZ1.1 (+), J1.10 (BUZZ1)
- new net: BZ1.2 (-), J1.12 (BUZZ2)
- no-connect marks 5 -> 3

Commit message: Drawt of PCB
Parts:
- BT1: footprint (none) -> local:Power_Port
- BZ1: footprint (none) -> Buzzer_Beeper:Buzzer_12x9.5RM7.6
- DS1: footprint (none) -> local:Screen_Port
- J1: footprint (none) -> local:Edge_Connector_Slot
- SW1, SW2, SW3, SW4, SW5, SW6, SW7, SW8, SW9: footprint (none) -> Button_Switch_THT:SW_PUSH_6mm_H5mm
- SW10: footprint (none) -> local:Power_Switch
Changed lines of the file:
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@@
 			)
 		)
-		(property "Footprint" ""
+		(property "Footprint" "Button_Switch_THT:SW_PUSH_6mm_H5mm"
 			(at 93.98 92.71 0)
 			(effects
@@
 			)
 		)
-		(property "Footprint" ""
+		(property "Footprint" "Button_Switch_THT:SW_PUSH_6mm_H5mm"
 			(at 132.08 80.01 0)
 			(effects
@@
 			)
 		)
-		(property "Footprint" ""
+		(property "Footprint" "Buzzer_Beeper:Buzzer_12x9.5RM7.6"
 			(at 268.605 83.82 90)
 			(effects
@@
 			)
 		)
-		(property "Footprint" ""
+		(property "Footprint" "Button_Switch_THT:SW_PUSH_6mm_H5mm"
 			(at 106.68 116.84 0)
 			(effects
@@
 			)
 		)
-		(property "Footprint" ""
+		(property "Footprint" "local:Power_Switch"
 			(at 90.17 166.37 0)
 			(effects
@@
 			)
 		)
-		(property "Footprint" ""
+		(property "Footprint" "Button_Switch_THT:SW_PUSH_6mm_H5mm"
 			(at 81.28 80.01 0)
 			(effects
@@
 			)
 		)
-		(property "Footprint" ""
+		(property "Footprint" "Button_Switch_THT:SW_PUSH_6mm_H5mm"
 			(at 68.58 92.71 0)
 			(effects
@@
 			)
 		)
-		(property "Footprint" ""
+		(property "Footprint" "local:Edge_Connector_Slot"
 			(at 223.52 92.71 0)
 			(effects
@@
 			)
 		)
-		(property "Footprint" ""
+		(property "Footprint" "Button_Switch_THT:SW_PUSH_6mm_H5mm"
 			(at 132.08 105.41 0)
 			(effects
@@
 			)
 		)
-		(property "Footprint" ""
+		(property "Footprint" "Button_Switch_THT:SW_PUSH_6mm_H5mm"
 			(at 119.38 92.71 0)
 			(effects
@@
 			)
 		)
-		(property "Footprint" ""
+		(property "Footprint" "local:Screen_Port"
 			(at 109.22 43.18 0)
 			(effects
@@
 			)
 		)
-		(property "Footprint" ""
+		(property "Footprint" "Button_Switch_THT:SW_PUSH_6mm_H5mm"
 			(at 81.28 105.41 0)
 			(effects
@@
 			)
 		)
-		(property "Footprint" ""
+		(property "Footprint" "Button_Switch_THT:SW_PUSH_6mm_H5mm"
 			(at 144.78 92.71 0)
 			(effects
@@
 			)
 		)
-		(property "Footprint" ""
+		(property "Footprint" "local:Power_Port"
 			(at 72.644 166.37 90)
 			(effects

Commit message: Add buzzer switch, separete baterry connectors, further PCD development
Parts:
- removed BT1: Battery, local:Power_Port, symbol Device:Battery
- added J2: -, local:Power_Port_Single_Minus, symbol Connector_Generic:Conn_01x01
- added J3: +, local:Power_Port_Single_Plus, symbol Connector_Generic:Conn_01x01
- added SW11: Buzzer_Switch, local:Power_Switch, symbol Switch:SW_DIP_x01
Connections:
- net GND: now also J2.1 (Pin_1)
- net at BZ1.1 (+): now also SW11.2; no longer J1.10 (BUZZ1)
- net at SW10.1: now also J3.1 (Pin_1)
- new net: J1.10 (BUZZ1), SW11.1
Other:
- moved on the sheet: BZ1, SW10
