File: Hardware/arducart/arducart.kicad_sch (KiCad schematic)
At the start: 0 parts

Commit message: First draft of ArduCart schematic
Parts:
- added J1: ~, symbol carts:Edge_Connector
- added J2: AVR-ISP-6, symbol Connector:AVR-ISP-6
- added R1, R2, R3, R4, R5, R6, R7, R8: 10k, symbol Device:R
- added U1: ~, symbol carts:Arduino_Pro_Mini
Connections:
- new net: J1.9 (BTN_MENU1), R1.2
- new net BTN_A: J1.21 (BTN_A1), J1.25 (BTN_X1), R2.2, U1.7 (D3)
- new net BTN_B: J1.22 (BTN_B1), J1.26 (BTN_Y1), R7.2, U1.8 (D2)
- new net BTN_DOWN: J1.14 (BTN_DOWN1), R4.2, U1.25 (A1)
- new net BTN_LEFT: J1.17 (BTN_LEFT1), R5.2, U1.24 (A2)
- new net BTN_RIGHT: J1.18 (BTN_RIGHT1), R6.2, U1.23 (A3)
- new net BTN_UP: J1.13 (BTN_UP1), R3.2, U1.26 (A0)
- new net BUZZER: J1.10 (BUZZ[+]), U1.2 (D8)
- new net GND: J1.11 (BTN_MENU2), J1.12 (BUZZ[-]), J1.15 (BTN_UP2), J1.16 (BTN_DOWN2), J1.19 (BTN_LEFT2), J1.20 (BTN_RIGHT2), J1.23 (BTN_A2), J1.24 (BTN_B2), J1.27 (BTN_X2), J1.28 (BTN_Y2), J1.29 (GND), J2.6 (GND), U1.20 (GND)
- new net ISP_MISO: J2.1 (MISO), U1.28 (D12(MISO))
- new net ISP_MOSI: J1.3 (SCR_SDA), J2.4 (MOSI), U1.29 (D11(MOSI))
- new net ISP_RST: J2.5 (~{RST}), R8.2, U1.10 (Reset)
- new net ISP_SCK: J1.5 (SCR_SCL), J2.3 (SCK), U1.27 (D13(SCK))
- new net SCREEN_DC: J1.8 (SCR_DC), U1.3 (D7)
- new net SCREEN_RESET: J1.6 (SCR_RES), U1.6 (D4)
- new net SPI_CS: J1.4 (SCR_CS), U1.4 (D6)
- new net VCC: J1.1 (VCC), J2.2 (VCC), R1.1, R2.1, R3.1, R4.1, R5.1, R6.1, R7.1, R8.1, U1.22 (VCC)
- no-connect marks 0 -> 22

Commit message: First draft of PCB design
Parts:
- J1: footprint (none) -> carts:Edge_Connector
- J2: footprint (none) -> Connector_PinHeader_2.54mm:PinHeader_2x03_P2.54mm_Horizontal
- R1, R2, R3, R4, R5, R6, R7, R8: footprint (none) -> Resistor_SMD:R_1206_3216Metric_Pad1.30x1.75mm_HandSolder
- U1: footprint (none) -> carts:Arduino_Pro_Mini
Changed lines of the file:
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@@
 			)
 		)
-		(property "Footprint" ""
+		(property "Footprint" "Resistor_SMD:R_1206_3216Metric_Pad1.30x1.75mm_HandSolder"
 			(at 163.322 64.77 90)
 			(effects
@@
 			)
 		)
-		(property "Footprint" ""
+		(property "Footprint" "Resistor_SMD:R_1206_3216Metric_Pad1.30x1.75mm_HandSolder"
 			(at 256.032 50.8 90)
 			(effects
@@
 			)
 		)
-		(property "Footprint" ""
+		(property "Footprint" "Resistor_SMD:R_1206_3216Metric_Pad1.30x1.75mm_HandSolder"
 			(at 26.162 90.17 90)
 			(effects
@@
 			)
 		)
-		(property "Footprint" ""
+		(property "Footprint" "Resistor_SMD:R_1206_3216Metric_Pad1.30x1.75mm_HandSolder"
 			(at 245.872 50.8 90)
 			(effects
@@
 			)
 		)
-		(property "Footprint" ""
+		(property "Footprint" "carts:Edge_Connector"
 			(at 73.66 104.14 0)
 			(effects
@@
 			)
 		)
-		(property "Footprint" ""
+		(property "Footprint" "Resistor_SMD:R_1206_3216Metric_Pad1.30x1.75mm_HandSolder"
 			(at 235.712 50.8 90)
 			(effects
@@
 			)
 		)
-		(property "Footprint" ""
+		(property "Footprint" "Resistor_SMD:R_1206_3216Metric_Pad1.30x1.75mm_HandSolder"
 			(at 145.542 64.77 90)
 			(effects
@@
 			)
 		)
-		(property "Footprint" ""
+		(property "Footprint" "Connector_PinHeader_2.54mm:PinHeader_2x03_P2.54mm_Horizontal"
 			(at 189.23 134.62 90)
 			(effects
@@
 			)
 		)
-		(property "Footprint" ""
+		(property "Footprint" "Resistor_SMD:R_1206_3216Metric_Pad1.30x1.75mm_HandSolder"
 			(at 154.432 64.77 90)
 			(effects
@@
 			)
 		)
-		(property "Footprint" ""
+		(property "Footprint" "Resistor_SMD:R_1206_3216Metric_Pad1.30x1.75mm_HandSolder"
 			(at 225.552 50.8 90)
 			(effects
@@
 			)
 		)
-		(property "Footprint" ""
+		(property "Footprint" "carts:Arduino_Pro_Mini"
 			(at 193.04 72.39 0)
 			(effects
